File: schematic/F091RC-ILI9488-PINMAP/F091RC-ILI9488-PINMAP.kicad_sch (KiCad schematic)
At the start: 3 parts

Commit message: removed testing power pin and added alarm to schematic
Connections:
- net ALARM: now reaches F091RC.32 (Pin_32)
Other:
- company: (none) -> VMC
- title: (none) -> Pin Mapping F091RC and ILI9488 - Raymond Protocol
Changed lines of the file:
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@@
 	(generator_version "10.0")
 	(paper "A4")
+	(title_block
+		(title "Pin Mapping F091RC and ILI9488 - Raymond Protocol")
+		(date "2026-08-07")
+		(rev "1.1")
+		(company "VMC")
+	)
 	(text "Colours"
 		(exclude_from_sim no)
@@
 	(wire
 		(pts
+			(xy 52.07 132.08) (xy 58.42 132.08)
+		)
+		(stroke
+			(width 0)
+			(type default)
+		)
+	)
+	(wire
+		(pts
 			(xy 21.59 114.3) (xy 39.37 114.3)
 		)
@@
 			)
 			(justify left bottom)
+		)
+	)
+	(label "ALARM"
+		(at 58.42 132.08 0)
+		(effects
+			(font
+				(size 1.27 1.27)
+				(color 255 153 0 1)
+			)
+			(justify left bottom)
